Commit message: (+) Added gazebo simulation

File: urdf/solid_robot.urdf.xacro (robot description, xacro)
@@ -1,4 +1,5 @@
 <?xml version="1.0"?>
 <robot xmlns:xacro="http://www.ros.org/wiki/xacro" name="solid_robot">
+    <link name="world" />
     <link name="base_link">
         <inertial>
@@ -40,4 +41,10 @@
         </collision>
     </link>
+    <joint
+        name="virtual_joint" type="fixed">
+        <parent link="world" />
+        <child link="base_link"/>
+        <origin rpy="0 0 0" xyz="0 0 0" />
+    </joint>
     <link name="link1">
         <inertial>
